File: KiCad/RV-8 electrical.sch (KiCad schematic (older format))
At the start: 20 parts

Commit message: Add new sheet for busses; replace generic symbols on backbone with sheet refs and labels
Parts:
- removed F? (x4): Fuse, symbol Device:Fuse
Connections:
- net labels added: B0, B1, E0, E1, M0, M1, M2
- wire segments 45 -> 47
Other:
- note removed: "BATT BUS"
- note removed: "ESS BUS"
- note removed: "MAIN BUS"
- moved on the sheet: D?, E_BUS_ALT_FEED, START, START_ARM
